File: 02_AMP/amp.kicad_pcb (KiCad board)
At the start: 2 copper layers, 63 x 53.5 mm, 27 parts, among them J1 Screw_Terminal_01x03, J2 Screw_Terminal_01x02, J3 Screw_Terminal_01x02, U1 LM1875

Commit message: C1裏面に予備パッド #3
Parts:
- added C7: 2.2u, Capacitor_SMD:C_1206_3216Metric, B.Cu at (158.9, 106.0)
Connections:
- TP5 pad 1: GND -> unconnected-(TP5-Pad1)
Routing:
- net Vin: track 24.2 -> 25.8 mm, vias 0 -> 1
- net Vin_AC: track 23.5 -> 25.0 mm, vias 0 -> 1
Other:
- board text added: "C1"
Changed lines of the file:
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@@
   (net 8 "Net-(R4-Pad2)")
   (net 9 "Vin_AC")
+  (net 10 "unconnected-(TP5-Pad1)")
   (footprint "TerminalBlock:TerminalBlock_bornier-2_P5.08mm" (layer "F.Cu")
     (at 195.326 113.411 90)
@@
     (property "ki_keywords" "test point tp")
     (attr exclude_from_pos_files)
-    (fp_text reference "TP4" (at 0 -2.148) (layer "F.SilkS") hide
+    (fp_text reference "TP4" (at 0 -2.148) (layer "F.SilkS")
         (effects (font (size 1 1) (thickness 0.15)))
     )
-    (fp_text value "GND" (at 0 2.25) (layer "F.SilkS")
+    (fp_text value "GND" (at 0 2.25) (layer "F.Fab")
         (effects (font (size 1 1) (thickness 0.15)))
     )
@@
     (property "ki_keywords" "test point tp")
     (attr exclude_from_pos_files)
-    (fp_text reference "TP2" (at 0 -2.148) (layer "F.SilkS") hide
+    (fp_text reference "TP2" (at 0 -2.148) (layer "F.SilkS")
         (effects (font (size 1 1) (thickness 0.15)))
     )
-    (fp_text value "Vin_AC" (at 0 2.25) (layer "F.SilkS")
+    (fp_text value "Vin_AC" (at 0 2.25) (layer "F.Fab")
         (effects (font (size 1 1) (thickness 0.15)))
     )
@@
     (property "ki_keywords" "test point tp")
     (attr exclude_from_pos_files)
-    (fp_text reference "TP6" (at 0 -2.148) (layer "F.SilkS") hide
+    (fp_text reference "TP6" (at 0 -2.148) (layer "F.SilkS")
         (effects (font (size 1 1) (thickness 0.15)))
     )
-    (fp_text value "GND" (at 0 2.25) (layer "F.SilkS")
+    (fp_text value "GND" (at 0 2.25) (layer "F.Fab")
         (effects (font (size 1 1) (thickness 0.15)))
     )
@@
     (property "ki_keywords" "test point tp")
     (attr exclude_from_pos_files)
-    (fp_text reference "TP3" (at 0 -2.148) (layer "F.SilkS") hide
+    (fp_text reference "TP3" (at 0 -2.148) (layer "F.SilkS")
         (effects (font (size 1 1) (thickness 0.15)))
     )
-    (fp_text value "Vout" (at 0 2.25) (layer "F.SilkS")
+    (fp_text value "Vout" (at 0 2.25) (layer "F.Fab")
         (effects (font (size 1 1) (thickness 0.15)))
     )
@@
     (property "ki_keywords" "test point tp")
     (attr exclude_from_pos_files)
-    (fp_text reference "TP1" (at 0 -2.148) (layer "F.SilkS") hide
+    (fp_text reference "TP1" (at 0 -2.148) (layer "F.SilkS")
         (effects (font (size 1 1) (thickness 0.15)))
     )
-    (fp_text value "Vin" (at 0 2.25) (layer "F.SilkS")
+    (fp_text value "Vin" (at 0 2.25) (layer "F.Fab")
         (effects (font (size 1 1) (thickness 0.15)))
     )
@@
     (property "ki_keywords" "test point tp")
     (attr exclude_from_pos_files)
-    (fp_text reference "TP5" (at 0 -2.148) (layer "F.SilkS") hide
+    (fp_text reference "TP5" (at 0 -2.148) (layer "F.SilkS")
         (effects (font (size 1 1) (thickness 0.15)))
     )
-    (fp_text value "GND" (at 3.556 0) (layer "F.SilkS")
+    (fp_text value "GND" (at 0 2.25) (layer "F.Fab")
         (effects (font (size 1 1) (thickness 0.15)))
     )
@@
       (stroke (width 0.05) (type solid)) (fill none) (layer "F.CrtYd"))
     (pad "1" thru_hole circle (at 0 0) (size 2.5 2.5) (drill 1.2) (layers "*.Cu" "*.Mask")
-      (net 3 "GND") (pinfunction "1") (pintype "passive"))
+      (net 10 "unconnected-(TP5-Pad1)") (pinfunction "1") (pintype "passive"))
   )
   (footprint "Heatsink:Heatsink_Fischer_SK129-STS_42x25mm_2xDrill2.5mm" (layer "F.Cu")
@@
     )
   )
+  (footprint "Capacitor_SMD:C_1206_3216Metric" (layer "B.Cu")
+    (at 158.877 105.967 -90)
+    (descr "Capacitor SMD 1206 (3216 Metric), square (rectangular) end terminal, IPC_7351 nominal, (Body size source: IPC-SM-782 page 76, https://www.pcb-3d.com/wordpress/wp-content/uploads/ipc-sm-782a_amendment_1_and_2.pdf), generated with kicad-footprint-generator")
+    (tags "capacitor")
+    (property "Sheetfile" "amp.kicad_sch")
+    (property "Sheetname" "")
+    (property "ki_description" "Unpolarized capacitor")
+    (property "ki_keywords" "cap capacitor")
+    (attr smd)
+    (fp_text reference "C7" (at 0 1.85 90) (layer "B.SilkS") hide
+        (effects (font (size 1 1) (thickness 0.15)) (justify mirror))
+    )
+    (fp_text value "2.2u" (at 0 -1.85 90) (layer "B.Fab")
+        (effects (font (size 1 1) (thickness 0.15)) (justify mirror))
+    )
+    (fp_text user "${REFERENCE}" (at 0 0 90) (layer "B.Fab")
+        (effects (font (size 0.8 0.8) (thickness 0.12)) (justify mirror))
+    )
+    (fp_line (start -0.711252 -0.91) (end 0.711252 -0.91)
+      (stroke (width 0.12) (type solid)) (layer "B.SilkS"))
+    (fp_line (start -0.711252 0.91) (end 0.711252 0.91)
+      (stroke (width 0.12) (type solid)) (layer "B.SilkS"))
+    (fp_line (start -2.3 -1.15) (end -2.3 1.15)
+      (stroke (width 0.05) (type solid)) (layer "B.CrtYd"))
+    (fp_line (start -2.3 1.15) (end 2.3 1.15)
+      (stroke (width 0.05) (type solid)) (layer "B.CrtYd"))
+    (fp_line (start 2.3 -1.15) (end -2.3 -1.15)
+      (stroke (width 0.05) (type solid)) (layer "B.CrtYd"))
+    (fp_line (start 2.3 1.15) (end 2.3 -1.15)
+      (stroke (width 0.05) (type solid)) (layer "B.CrtYd"))
+    (fp_line (start -1.6 -0.8) (end -1.6 0.8)
+      (stroke (width 0.1) (type solid)) (layer "B.Fab"))
+    (fp_line (start -1.6 0.8) (end 1.6 0.8)
+      (stroke (width 0.1) (type solid)) (layer "B.Fab"))
+    (fp_line (start 1.6 -0.8) (end -1.6 -0.8)
+      (stroke (width 0.1) (type solid)) (layer "B.Fab"))
+    (fp_line (start 1.6 0.8) (end 1.6 -0.8)
+      (stroke (width 0.1) (type solid)) (layer "B.Fab"))
+    (pad "1" smd roundrect (at -1.475 0 270) (size 1.15 1.8) (layers "B.Cu" "B.Paste" "B.Mask") (roundrect_rratio 0.217391)
+      (net 1 "Vin") (pintype "passive"))
+    (pad "2" smd roundrect (at 1.475 0 270) (size 1.15 1.8) (layers "B.Cu" "B.Paste" "B.Mask") (roundrect_rratio 0.217391)
+      (net 9 "Vin_AC") (pintype "passive"))
+    (model "${KICAD6_3DMODEL_DIR}/Capacitor_SMD.3dshapes/C_1206_3216Metric.wrl"
+      (offset (xyz 0 0 0))
+      (scale (xyz 1 1 1))
+      (rotate (xyz 0 0 0))
+    )
+  )
   (gr_poly
     (pts
@@
   (gr_arc (start 146.812 129.286) (mid 144.297528 128.244472) (end 143.256 125.73)
     (stroke (width 0.1) (type default)) (layer "Edge.Cuts"))
+  (gr_text "C1" (at 159.004 109.601 90) (layer "B.SilkS")
+    (effects (font (size 1 1) (thickness 0.15)) (justify mirror))
+  )
   (gr_text "アンプ基板" (at 189.738 127.508) (layer "F.SilkS")
     (effects (font (face "BIZ UDゴシック") (size 1.8 1.8) (thickness 0.15)) (justify bottom))
@@
     )
   )
+  (segment (start 157.544 105.22) (end 156.591 105.22) (width 0.5) (layer "F.Cu") (net 1))
   (segment (start 158.305 105.22) (end 158.955 104.57) (width 0.5) (layer "F.Cu") (net 1))
   (segment (start 151.701 100.33) (end 149.733 100.33) (width 0.5) (layer "F.Cu") (net 1))
   (segment (start 149.733 100.33) (end 154.305 95.758) (width 0.5) (layer "F.Cu") (net 1))
+  (segment (start 157.544 105.22) (end 158.305 105.22) (width 0.5) (layer "F.Cu") (net 1))
   (segment (start 154.305 95.758) (end 154.305 89.535) (width 0.5) (layer "F.Cu") (net 1))
-  (segment (start 156.591 105.22) (end 158.305 105.22) (width 0.5) (layer "F.Cu") (net 1))
   (segment (start 156.591 105.22) (end 151.701 100.33) (width 0.5) (layer "F.Cu") (net 1))
+  (via (at 157.544 105.22) (size 0.8) (drill 0.4) (layers "F.Cu" "B.Cu") (net 1))
+  (segment (start 158.149 105.22) (end 158.877 104.492) (width 0.5) (layer "B.Cu") (net 1))
+  (segment (start 157.544 105.22) (end 158.149 105.22) (width 0.5) (layer "B.Cu") (net 1))
   (segment (start 181.229 104.59) (end 181.2 104.619) (width 2) (layer "F.Cu") (net 2))
   (segment (start 181.2 97.376) (end 181.229 97.405) (width 2) (layer "F.Cu") (net 2))
@@
   (segment (start 176.721 109.982) (end 177.8 111.061) (width 0.5) (layer "F.Cu") (net 8))
   (segment (start 173.672 109.982) (end 176.721 109.982) (width 0.5) (layer "F.Cu") (net 8))
+  (segment (start 160.352 107.52) (end 158.955 107.52) (width 0.5) (layer "F.Cu") (net 9))
   (segment (start 160.64 107.52) (end 161.29 106.87) (width 0.5) (layer "F.Cu") (net 9))
-  (segment (start 158.955 107.52) (end 160.64 107.52) (width 0.5) (layer "F.Cu") (net 9))
   (segment (start 165.481 107.445) (end 165.481 110.49) (width 0.5) (layer "F.Cu") (net 9))
   (segment (start 164.906 106.87) (end 174.4 97.376) (width 0.5) (layer "F.Cu") (net 9))
   (segment (start 161.29 106.87) (end 164.906 106.87) (width 0.5) (layer "F.Cu") (net 9))
+  (segment (start 160.352 107.52) (end 160.64 107.52) (width 0.5) (layer "F.Cu") (net 9))
   (segment (start 164.906 106.87) (end 165.481 107.445) (width 0.5) (layer "F.Cu") (net 9))
+  (via (at 160.352 107.52) (size 0.8) (drill 0.4) (layers "F.Cu" "B.Cu") (net 9))
+  (segment (start 158.955 107.52) (end 158.877 107.442) (width 0.5) (layer "B.Cu") (net 9))
+  (segment (start 160.352 107.52) (end 158.955 107.52) (width 0.5) (layer "B.Cu") (net 9))
   (zone (net 3) (net_name "GND") (layers "F&B.Cu") (hatch edge 0.5)
     (connect_pads (clearance 0.5))
