File: 02_AMP/amp.kicad_sch (KiCad schematic)
At the start: 18 parts, among them J1 Screw_Terminal_01x03, J2 Screw_Terminal_01x02, U1 LM1875

Commit message: 部品仮配置
Parts:
- added J3: Screw_Terminal_01x02, TerminalBlock:TerminalBlock_bornier-2_P5.08mm, symbol Connector:Screw_Terminal_01x02
- added TP4, TP5, TP6: GND, TestPoint_THTPad_D2.5mm_Drill1.2mm, symbol Connector:TestPoint
Connections:
- net GND: now also J3.1 (Pin_1), TP4.1, TP6.1
- net Vin: now also J3.2 (Pin_2)
- net Vin_AC: now reaches C1.2, R2.1, TP2.1, U1.1 (+)
Changed lines of the file:
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@@
   (junction (at 99.695 80.01) (diameter 0) (color 0 0 0 0)
   )
+  (junction (at 71.755 103.505) (diameter 0) (color 0 0 0 0)
+  )
   (junction (at 135.255 114.935) (diameter 0) (color 0 0 0 0)
   )
@@
     (stroke (width 0) (type default))
   )
+  (wire (pts (xy 71.755 103.505) (xy 71.755 104.775))
+    (stroke (width 0) (type default))
+  )
   (wire (pts (xy 106.045 60.96) (xy 113.665 60.96))
     (stroke (width 0) (type default))
@@
   )
   (wire (pts (xy 83.82 90.805) (xy 83.82 93.345))
+    (stroke (width 0) (type default))
+  )
+  (wire (pts (xy 78.105 103.505) (xy 71.755 103.505))
     (stroke (width 0) (type default))
   )
@@
   (text "可変抵抗実装用" (at 127 123.825 0)
     (effects (font (face "BIZ UDゴシック") (size 1.27 1.27)) (justify left bottom))
+  )
+  (global_label "Vin" (shape input) (at 63.5 91.44 0) (fields_autoplaced)
+    (effects (font (size 1.27 1.27)) (justify left))
+    (property "Intersheetrefs" "${INTERSHEET_REFS}" (at 69.3276 91.44 0)
+      (effects (font (size 1.27 1.27)) (justify left) hide)
+    )
   )
   (global_label "Vout" (shape input) (at 161.29 91.44 180) (fields_autoplaced)
@@
     )
   )
+  (global_label "Vin_AC" (shape input) (at 96.52 80.01 90) (fields_autoplaced)
+    (effects (font (size 1.27 1.27)) (justify left))
+    (property "Intersheetrefs" "${INTERSHEET_REFS}" (at 96.52 70.8562 90)
+      (effects (font (size 1.27 1.27)) (justify left) hide)
+    )
+  )
   (global_label "-30V" (shape input) (at 115.57 92.075 0) (fields_autoplaced)
     (effects (font (size 1.27 1.27)) (justify left))
@@
     )
   )
+  (symbol (lib_id "power:GND") (at 71.755 104.775 0) (unit 1)
+    (in_bom yes) (on_board yes) (dnp no) (fields_autoplaced)
+    (property "Reference" "#PWR011" (at 71.755 111.125 0)
+      (effects (font (size 1.27 1.27)) hide)
+    )
+    (property "Value" "GND" (at 71.755 109.22 0)
+      (effects (font (size 1.27 1.27)))
+    )
+    (property "Footprint" "" (at 71.755 104.775 0)
+      (effects (font (size 1.27 1.27)) hide)
+    )
+    (property "Datasheet" "" (at 71.755 104.775 0)
+      (effects (font (size 1.27 1.27)) hide)
+    )
+    (pin "1")
+    (instances
+      (project "amp"
+        (path "/d7b1d85c-c305-4915-b769-ec0537650afa"
+          (reference "#PWR011") (unit 1)
+        )
+      )
+    )
+  )
   (symbol (lib_id "Device:R") (at 130.175 114.935 90) (unit 1)
     (in_bom yes) (on_board yes) (dnp no) (fields_autoplaced)
@@
     )
   )
+  (symbol (lib_id "Connector:TestPoint") (at 74.723 103.5924 0) (unit 1)
+    (in_bom yes) (on_board yes) (dnp no) (fields_autoplaced)
+    (property "Reference" "TP5" (at 76.628 99.0204 0)
+      (effects (font (size 1.27 1.27)) (justify left))
+    )
+    (property "Value" "GND" (at 76.628 101.5604 0)
+      (effects (font (size 1.27 1.27)) (justify left))
+    )
+    (property "Footprint" "TestPoint_THTPad_D2.5mm_Drill1.2mm" (at 79.803 103.5924 0)
+      (effects (font (size 1.27 1.27)) hide)
+    )
+    (property "Datasheet" "~" (at 79.803 103.5924 0)
+      (effects (font (size 1.27 1.27)) hide)
+    )
+    (pin "1")
+    (instances
+      (project "amp"
+        (path "/d7b1d85c-c305-4915-b769-ec0537650afa"
+          (reference "TP5") (unit 1)
+        )
+      )
+    )
+  )
+  (symbol (lib_id "power:GND") (at 63.5 93.98 0) (unit 1)
+    (in_bom yes) (on_board yes) (dnp no) (fields_autoplaced)
+    (property "Reference" "#PWR010" (at 63.5 100.33 0)
+      (effects (font (size 1.27 1.27)) hide)
+    )
+    (property "Value" "GND" (at 63.5 98.425 0)
+      (effects (font (size 1.27 1.27)))
+    )
+    (property "Footprint" "" (at 63.5 93.98 0)
+      (effects (font (size 1.27 1.27)) hide)
+    )
+    (property "Datasheet" "" (at 63.5 93.98 0)
+      (effects (font (size 1.27 1.27)) hide)
+    )
+    (pin "1")
+    (instances
+      (project "amp"
+        (path "/d7b1d85c-c305-4915-b769-ec0537650afa"
+          (reference "#PWR010") (unit 1)
+        )
+      )
+    )
+  )
   (symbol (lib_id "Connector:TestPoint") (at 132.715 82.55 0) (unit 1)
     (in_bom yes) (on_board yes) (dnp no) (fields_autoplaced)
@@
         (path "/d7b1d85c-c305-4915-b769-ec0537650afa"
           (reference "R1") (unit 1)
+        )
+      )
+    )
+  )
+  (symbol (lib_id "Connector:TestPoint") (at 78.105 103.505 0) (unit 1)
+    (in_bom yes) (on_board yes) (dnp no) (fields_autoplaced)
+    (property "Reference" "TP6" (at 80.01 98.933 0)
+      (effects (font (size 1.27 1.27)) (justify left))
+    )
+    (property "Value" "GND" (at 80.01 101.473 0)
+      (effects (font (size 1.27 1.27)) (justify left))
+    )
+    (property "Footprint" "TestPoint_THTPad_D2.5mm_Drill1.2mm" (at 83.185 103.505 0)
+      (effects (font (size 1.27 1.27)) hide)
+    )
+    (property "Datasheet" "~" (at 83.185 103.505 0)
+      (effects (font (size 1.27 1.27)) hide)
+    )
+    (pin "1")
+    (instances
+      (project "amp"
+        (path "/d7b1d85c-c305-4915-b769-ec0537650afa"
+          (reference "TP6") (unit 1)
         )
       )
@@
         )
       )
+    )
+  )
+  (symbol (lib_id "Connector:Screw_Terminal_01x02") (at 58.42 93.98 180) (unit 1)
+    (in_bom yes) (on_board yes) (dnp no) (fields_autoplaced)
+    (property "Reference" "J3" (at 58.42 85.725 0)
+      (effects (font (size 1.27 1.27)))
+    )
+    (property "Value" "Screw_Terminal_01x02" (at 58.42 88.265 0)
+      (effects (font (size 1.27 1.27)))
+    )
+    (property "Footprint" "TerminalBlock:TerminalBlock_bornier-2_P5.08mm" (at 58.42 93.98 0)
+      (effects (font (size 1.27 1.27)) hide)
+    )
+    (property "Datasheet" "~" (at 58.42 93.98 0)
+      (effects (font (size 1.27 1.27)) hide)
+    )
+    (pin "1")
+    (pin "2")
+    (instances
+      (project "amp"
+        (path "/d7b1d85c-c305-4915-b769-ec0537650afa"
+          (reference "J3") (unit 1)
+        )
+      )
+    )
+  )
+  (symbol (lib_id "Connector:TestPoint") (at 71.755 103.505 0) (unit 1)
+    (in_bom yes) (on_board yes) (dnp no) (fields_autoplaced)
+    (property "Reference" "TP4" (at 73.66 98.933 0)
+      (effects (font (size 1.27 1.27)) (justify left))
+    )
+    (property "Value" "GND" (at 73.66 101.473 0)
+      (effects (font (size 1.27 1.27)) (justify left))
+    )
+    (property "Footprint" "TestPoint_THTPad_D2.5mm_Drill1.2mm" (at 76.835 103.505 0)
+      (effects (font (size 1.27 1.27)) hide)
+    )
+    (property "Datasheet" "~" (at 76.835 103.505 0)
+      (effects (font (size 1.27 1.27)) hide)
+    )
+    (pin "1")
+    (instances
+      (project "amp"
+        (path "/d7b1d85c-c305-4915-b769-ec0537650afa"
+          (reference "TP4") (unit 1)
+        )
+      )

Commit message: C1裏面に予備パッド #3
Parts:
- added C7: 2.2u, Capacitor_SMD:C_1206_3216Metric, symbol Device:C
Connections:
- net Vin: now also C7.1
- net Vin_AC: now also C7.2
Changed lines of the file:
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@@
   (junction (at 132.715 82.55) (diameter 0) (color 0 0 0 0)
   )
+  (junction (at 88.265 80.01) (diameter 0) (color 0 0 0 0)
+  )
   (junction (at 113.665 95.25) (diameter 0) (color 0 0 0 0)
   )
@@
   (junction (at 138.43 82.55) (diameter 0) (color 0 0 0 0)
   )
+  (junction (at 95.885 80.01) (diameter 0) (color 0 0 0 0)
+  )
   (wire (pts (xy 98.425 90.805) (xy 98.425 93.345))
     (stroke (width 0) (type default))
@@
     (stroke (width 0) (type default))
   )
+  (wire (pts (xy 95.885 80.01) (xy 95.885 85.09))
+    (stroke (width 0) (type default))
+  )
   (wire (pts (xy 138.43 82.55) (xy 132.715 82.55))
     (stroke (width 0) (type default))
@@
   )
   (wire (pts (xy 78.105 80.01) (xy 80.645 80.01))
+    (stroke (width 0) (type default))
+  )
+  (wire (pts (xy 88.265 85.09) (xy 88.265 80.01))
     (stroke (width 0) (type default))
   )
@@
         )
       )
+    )
+  )
+  (symbol (lib_id "Device:C") (at 92.075 85.09 90) (unit 1)
+    (in_bom yes) (on_board yes) (dnp no) (fields_autoplaced)
+    (property "Reference" "C7" (at 92.075 77.47 90)
+      (effects (font (size 1.27 1.27)))
+    )
+    (property "Value" "2.2u" (at 92.075 80.01 90)
+      (effects (font (size 1.27 1.27)))
+    )
+    (property "Footprint" "Capacitor_SMD:C_1206_3216Metric" (at 95.885 84.1248 0)
+      (effects (font (size 1.27 1.27)) hide)
+    )
+    (property "Datasheet" "~" (at 92.075 85.09 0)
+      (effects (font (size 1.27 1.27)) hide)
+    )
+    (pin "1")
+    (pin "2")
+    (instances
+      (project "amp"
+        (path "/d7b1d85c-c305-4915-b769-ec0537650afa"
+          (reference "C7") (unit 1)
+        )
+      )
